File: schematics/src/ioboard/ioboard.sch (EAGLE design)
At the start: 36 parts, among them IC7 TL072P

Commit message: Fixed some bugs and updated documentation
Parts:
- R26: value 1.5k -> 3k
Changed lines of the file:
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@@
 <part name="R24" library="resistor" deviceset="R-US_" device="0204/7" value="2.2k"/>
 <part name="R25" library="resistor" deviceset="R-US_" device="0204/7" value="3k"/>
-<part name="R26" library="resistor" deviceset="R-US_" device="0204/7" value="1.5k"/>
+<part name="R26" library="resistor" deviceset="R-US_" device="0204/7" value="3k"/>
 <part name="R27" library="resistor" deviceset="R-US_" device="0204/7" value="180k"/>
 <part name="GND12" library="supply1" deviceset="GND" device=""/>
