File: schematics/src/mainboard/mainboard.brd (EAGLE design)
At the start: 48.3 x 99.1 mm, 73 parts, among them IC1 566, IC2 TL074P, IC4 4013N, IC5 TL072P, IC6 TL072P, Q1 2N3904, Q2 2N3906, Q3 2N3904, Q4 2N3904, Q5 BF245

Commit message: Updated Schematics, Fixed Power Socket orientation
Parts:
- removed C6, C7: 10uF, resistor:E2,5-5
- added C12, C19: 10uf, resistor:E2,5-5
- moved PWR 0.63 mm to (24.1, 5.71), turned to 180 degrees
Connections:
- net +12V: now also C19.+, PWR.10, PWR.9; no longer C7.+, PWR.1, PWR.2
- net -12V: now also C12.-, PWR.1, PWR.2; no longer C6.-, PWR.10, PWR.9
- net GND: now also C12.+, C19.-; no longer C6.+, C7.-
Routing:
- net +12V: track 185.1 -> 186.6 mm
- net -12V: track 206.5 -> 205.1 mm
- net SQR_OUT: vias 1 -> 0

Commit message: Fixed minor issues, added documentation and updated some faceplates
Parts:
- turned C2 to 180 degrees
Connections:
- net -12V: now also C2.-; no longer C2.+
- net GND: now also C2.+; no longer C2.-
Changed lines of the file:
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@@
 <attribute name="VALUE" x="24.765" y="16.129" size="1.27" layer="27" ratio="10" rot="R90"/>
 </element>
-<element name="C2" library="resistor" package="E2,5-6" value="4.7uF" x="33.02" y="15.875" smashed="yes">
-<attribute name="NAME" x="28.575" y="12.7" size="1.27" layer="25" font="vector" ratio="10"/>
-<attribute name="VALUE" x="35.687" y="13.208" size="1.27" layer="27" ratio="10"/>
+<element name="C2" library="resistor" package="E2,5-6" value="4.7uF" x="33.02" y="15.875" smashed="yes" rot="R180">
+<attribute name="NAME" x="37.465" y="19.05" size="1.27" layer="25" font="vector" ratio="10" rot="R180"/>
+<attribute name="VALUE" x="30.353" y="18.542" size="1.27" layer="27" ratio="10" rot="R180"/>
 </element>
 <element name="C3" library="resistor" package="C050-024X044" value=".047uF" x="17.145" y="15.875" smashed="yes" rot="R270">
@@
 <signal name="GND" airwireshidden="yes">
 <contactref element="IC1" pad="8"/>
-<contactref element="C2" pad="-"/>
 <contactref element="R2" pad="1"/>
 <contactref element="R4" pad="1"/>
@@
 <contactref element="PWR" pad="6"/>
 <contactref element="C19" pad="-"/>
+<contactref element="C2" pad="+"/>
 <wire x1="38.735" y1="86.995" x2="45.72" y2="93.345" width="0" layer="19" extent="1-1"/>
 <wire x1="36.195" y1="79.375" x2="38.735" y2="86.995" width="0" layer="19" extent="1-1"/>
@@
 <wire x1="34.29" y1="15.875" x2="36.195" y2="20.955" width="0" layer="19" extent="1-1"/>
 <wire x1="37.465" y1="10.795" x2="34.29" y2="15.875" width="0" layer="19" extent="1-1"/>
+<wire x1="41.275" y1="5.715" x2="37.465" y2="10.795" width="0" layer="19" extent="1-1"/>
 <wire x1="20.955" y1="26.035" x2="27.94" y2="34.29" width="0" layer="19" extent="1-1"/>
 <wire x1="20.32" y1="15.875" x2="20.955" y2="26.035" width="0" layer="19" extent="1-1"/>
+<wire x1="21.59" y1="6.985" x2="20.32" y2="15.875" width="0" layer="19" extent="1-1"/>
+<wire x1="24.13" y1="6.985" x2="21.59" y2="6.985" width="0" layer="19" extent="1-1"/>
+<wire x1="26.67" y1="6.985" x2="24.13" y2="6.985" width="0" layer="19" extent="1-1"/>
+<wire x1="26.67" y1="4.445" x2="26.67" y2="6.985" width="0" layer="19" extent="1-1"/>
+<wire x1="24.13" y1="4.445" x2="24.13" y2="6.985" width="0" layer="19" extent="1-1"/>
+<wire x1="21.59" y1="4.445" x2="21.59" y2="6.985" width="0" layer="19" extent="1-1"/>
 <wire x1="9.525" y1="17.145" x2="20.32" y2="15.875" width="0" layer="19" extent="1-1"/>
 <wire x1="6.985" y1="13.97" x2="9.525" y2="17.145" width="0" layer="19" extent="1-1"/>
 <wire x1="2.54" y1="12.7" x2="6.985" y2="13.97" width="0" layer="19" extent="1-1"/>
 <wire x1="8.89" y1="24.13" x2="9.525" y2="17.145" width="0" layer="19" extent="1-1"/>
+<wire x1="6.985" y1="5.715" x2="6.985" y2="13.97" width="0" layer="19" extent="1-1"/>
 <wire x1="8.89" y1="34.29" x2="8.89" y2="24.13" width="0" layer="19" extent="1-1"/>
 <wire x1="10.16" y1="36.83" x2="8.89" y2="34.29" width="0" layer="19" extent="1-1"/>
@@
 <wire x1="20.32" y1="97.155" x2="27.94" y2="97.155" width="0" layer="19" extent="1-1"/>
 <wire x1="20.32" y1="92.075" x2="20.32" y2="97.155" width="0" layer="19" extent="1-1"/>
-<wire x1="26.67" y1="4.445" x2="2.54" y2="12.7" width="0" layer="19" extent="1-1"/>
-<wire x1="24.13" y1="4.445" x2="26.67" y2="4.445" width="0" layer="19" extent="1-1"/>
-<wire x1="21.59" y1="4.445" x2="24.13" y2="4.445" width="0" layer="19" extent="1-1"/>
-<wire x1="21.59" y1="6.985" x2="21.59" y2="4.445" width="0" layer="19" extent="1-1"/>
-<wire x1="24.13" y1="6.985" x2="24.13" y2="4.445" width="0" layer="19" extent="1-1"/>
-<wire x1="26.67" y1="6.985" x2="26.67" y2="4.445" width="0" layer="19" extent="1-1"/>
-<wire x1="6.985" y1="5.715" x2="21.59" y2="6.985" width="0" layer="19" extent="1-1"/>
-<wire x1="41.275" y1="5.715" x2="26.67" y2="6.985" width="0" layer="19" extent="1-1"/>
 </signal>
 <signal name="-12V">
 <contactref element="IC1" pad="1"/>
-<contactref element="C2" pad="+"/>
 <contactref element="C3" pad="2"/>
 <contactref element="R3" pad="2"/>
@@
 <wire x1="22.225" y1="36.83" x2="20.32" y2="36.83" width="0.6096" layer="16"/>
 <wire x1="15.24" y1="36.83" x2="20.32" y2="36.83" width="0.6096" layer="16"/>
-<wire x1="27.94" y1="15.875" x2="31.75" y2="15.875" width="0.6096" layer="1"/>
 <via x="24.765" y="36.195" extent="1-16" drill="0.35"/>
 <wire x1="27.94" y1="58.42" x2="24.765" y2="58.42" width="0.6096" layer="16"/>
@@
 <wire x1="29.21" y1="5.715" x2="29.21" y2="4.445" width="0.6096" layer="1"/>
 <wire x1="38.735" y1="5.715" x2="29.21" y2="5.715" width="0.6096" layer="1"/>
+<contactref element="C2" pad="-"/>
+<wire x1="27.94" y1="15.875" x2="31.75" y2="15.875" width="0.6096" layer="1"/>
 </signal>
 <signal name="N$1">

Commit message: Fixed some bugs and updated documentation
Parts:
- R32, R37: value 1.5k -> 3k
Changed lines of the file:
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@@
 <attribute name="VALUE" x="14.9606" y="70.9676" size="0.9906" layer="27" ratio="10" rot="R180"/>
 </element>
-<element name="R32" library="resistor" package="0204/7" value="1.5k" x="13.335" y="67.945" smashed="yes" rot="R180">
+<element name="R32" library="resistor" package="0204/7" value="3k" x="13.335" y="67.945" smashed="yes" rot="R180">
 <attribute name="NAME" x="11.43" y="67.31" size="0.9906" layer="25" font="vector" ratio="10"/>
 <attribute name="VALUE" x="14.9606" y="68.4276" size="0.9906" layer="27" ratio="10" rot="R180"/>
@@
 <attribute name="VALUE" x="33.2994" y="67.4624" size="0.9906" layer="27" ratio="10"/>
 </element>
-<element name="R37" library="resistor" package="0204/7" value="1.5k" x="34.925" y="65.405" smashed="yes">
+<element name="R37" library="resistor" package="0204/7" value="3k" x="34.925" y="65.405" smashed="yes">
 <attribute name="NAME" x="33.02" y="64.77" size="0.9906" layer="25" font="vector" ratio="10"/>
 <attribute name="VALUE" x="33.2994" y="64.9224" size="0.9906" layer="27" ratio="10"/>
